Commit message: see #1;

File: urdf/a1.urdf (robot description, URDF)
Before this commit: robot a1_description, 23 links, 22 joints
Links:
- link FL_thigh_shoulder: mass None -> 0.001
- link FR_thigh_shoulder: mass None -> 0.001
- link RL_thigh_shoulder: mass None -> 0.001
- link RR_thigh_shoulder: mass None -> 0.001
- link base: mass None -> 0.001
